Commit message: Modified a bit

File: config/models/ship1.urdf (robot description, URDF)
Before this commit: robot ship1, 1 links, 0 joints
Links:
- link obstacles/ship1: geometry visual mesh filename=package://asv_simulator/meshes/Revolt.STL scale=0.0001 0.0001 0.0001

File: config/models/simple.urdf (robot description, URDF)
Before this commit: robot asv, 1 links, 0 joints
Links:
- link asv: geometry visual mesh filename=package://asv_simulator/meshes/Revolt.STL scale=0.0001 0.0001 0.0001
