Commit message: Modified configurations

File: config/models/ship2.urdf (robot description, URDF)
Before this commit: robot ship1, 1 links, 0 joints
Links:
- removed link obstacles/ship1
- added link obstacles/ship2; visual mesh filename=package://asv_simulator/meshes/Revolt.STL scale=0.0001 0.0001 0.0001
